File: EFUSE2024/EFUSE2024.kicad_sch (KiCad schematic)
At the start: 22 parts, among them Q3 CSD19532Q5B, Q4 CSD19532Q5B, Q7 BSS138, U5 TPS26631PWP, U6 TPS26631PWP, U7 TPS26630RGE

Commit message: schematic
Parts:
- added C1, C10, C11, C12, C13, C14, C15, C9: C, symbol Device:C
- added R10, R11, R12, R13, R14, R9: R, symbol Device:R
- added U1, U2, U3: TPS26630RGE, Package_DFN_QFN:Texas_RGE0024H_VQFN-24-1EP_4x4mm_P0.5mm_EP2.7x2.7mm_ThermalVias, symbol Power_Management:TPS26630RGE
Connections:
- net at U7.1 (IN), U7.2 (IN): now also C1.1, C13.1, C15.1, C9.1, R9.1, U1.1 (IN), U1.2 (IN), U2.1 (IN), U2.2 (IN), U3.1 (IN), U3.2 (IN)
- net at U7.10 (ILIM): now also R12.1
- net at U7.11 (MODE): now also U7.25 (GND), U7.8 (GND), C11.2, R11.2, R12.2, R13.2
- net at U7.12 (~{SHDN}): now also U1.12 (~{SHDN}), U2.12 (~{SHDN})
- net at U7.13 (IMON): now also R13.1, U1.13 (IMON), U2.13 (IMON)
- net at U7.17 (OUT), U7.18 (OUT): now also C10.1, C12.1, C14.1, U1.17 (OUT), U1.18 (OUT), U2.17 (OUT), U2.18 (OUT), U3.17 (OUT), U3.18 (OUT)
- net at U7.6 (UVLO): now also R10.1, R9.2, U1.6 (UVLO), U2.6 (UVLO)
- net at U7.7 (OVP): now also R10.2, R11.1, U1.7 (OVP), U2.7 (OVP)
- net at U7.9 (dVdT): now also C11.1, U1.9 (dVdT), U2.9 (dVdT)
- new net: U3.25 (GND), U3.8 (GND)
- new net: R14.1, U1.10 (ILIM)
- new net: R14.2, U1.11 (MODE), U1.25 (GND), U1.8 (GND)
- new net: U2.25 (GND), U2.8 (GND)
Other:
- moved on the sheet: U7

Commit message: Adding to schematic
Parts:
- added C16, C17, C18: C, symbol Device:C
- added R15, R16: R, symbol Device:R
Connections:
- net GND: now also C1.2, C10.2, C11.2, C12.2, C13.2, C14.2, C15.2, C9.2, R11.2, R12.2, R13.2, R14.2, U1.11 (MODE), U1.25 (GND), U1.8 (GND), U2.11 (MODE), U2.25 (GND), U2.8 (GND), U3.11 (MODE), U3.25 (GND), U3.8 (GND), U7.11 (MODE), U7.25 (GND), U7.8 (GND), C16.2, C17.2, C18.2, R15.2, R16.2
- net at C1.1, C13.1, C15.1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: now also C16.1
- net at U1.12 (~{SHDN}), U2.12 (~{SHDN}), U7.12 (~{SHDN}): now also U3.12 (~{SHDN})
- net at R13.1, U1.13 (IMON), U2.13 (IMON)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: now also U3.13 (IMON)
- net at C10.1, C12.1, C14.1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: now also C17.1, C18.1
- net at R10.1, R9.2, U1.6 (UVLO)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: now also U3.6 (UVLO)
- net at R10.2, R11.1, U1.7 (OVP)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: now also U3.7 (OVP)
- net at C11.1, U1.9 (dVdT), U2.9 (dVdT)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: now also U3.9 (dVdT)
- net at U3.10 (ILIM): now also R16.1
- net at U2.10 (ILIM): now also R15.1
Other:
- moved on the sheet: C1, C11, C14, C2, C3, C4, C5, C6, C7, C8, D1, Q3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

Commit message: asjdflk
Parts:
- removed R14, R15, R16: R, symbol Device:R
- added RILIM1, RILIM2, RILIM3: 3.33kΩ, symbol Device:R
- C1, C10, C11, C12, C13, C14, C15, C16, C17, C18, C9: value C -> 0.1uF
- R1: renamed from R9; value R -> 887kΩ
- R2: renamed from R10; value R -> 29.4 kΩ
- R3: renamed from R11; value R -> 34kΩ
- RILIM: renamed from R12; value R -> 3.33kΩ
- RIMON: renamed from R13; value R -> 2.46kΩ
Connections:
- net GND: now also RILIM1.2, RILIM2.2, RILIM3.2
- net at U3.10 (ILIM): now also RILIM3.1
- net at U2.10 (ILIM): now also RILIM2.1
- net at U1.10 (ILIM): now also RILIM1.1

Commit message: deleted two
Parts:
- removed C2, C3, C4, C5, C6, C7, C8: 0.1uF, symbol Device:C
- removed D1: 1.5SMCxxCA, Diode_SMD:D_SMC, symbol Diode:1.5SMCxxCA
- removed Q3, Q4: CSD19532Q5B, Package_TO_SOT_SMD:TDSON-8-1, symbol Transistor_FET:CSD19532Q5B
- removed Q7: BSS138, Package_TO_SOT_SMD:SOT-23, symbol Transistor_FET:BSS138
- removed R1, R2, R3, R4, R5, R6, R7, R8: R, symbol Device:R
- removed U5, U6: TPS26631PWP, Package_SO:HTSSOP-20-1EP_4.4x6.5mm_P0.65mm_EP3.4x6.5mm_Mask2.96x2.96mm_ThermalVias, symbol Power_Management:TPS26631PWP

Commit message: added connector
Parts:
- added J1, J2: Conn_01x02_Pin, symbol Connector:Conn_01x02_Pin
Connections:
- net GND: now also J1.1 (Pin_1), J2.2 (Pin_2)
- net at C1.1, C13.1, C15.1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: now also J2.1 (Pin_1)
- net at C10.1, C12.1, C14.1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: now also J1.2 (Pin_2)

Commit message: Added footprints
Parts:
- C1, C10, C11, C12, C13, C14, C15, C16, C17, C18, C9, J1, J2: footprint (none) -> Capacitor_SMD:C_0805_2012Metric_Pad1.18x1.45mm_HandSolder
- R1, R2, R3, RILIM, RILIM1, RILIM2, RILIM3, RIMON: footprint (none) -> Resistor_SMD:R_0805_2012Metric_Pad1.20x1.40mm_HandSolder
Changed lines of the file:
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@@
 			)
 		)
-		(property "Footprint" ""
+		(property "Footprint" "Capacitor_SMD:C_0805_2012Metric_Pad1.18x1.45mm_HandSolder"
 			(at 26.3652 31.75 0)
 			(effects
@@
 			)
 		)
-		(property "Footprint" ""
+		(property "Footprint" "Capacitor_SMD:C_0805_2012Metric_Pad1.18x1.45mm_HandSolder"
 			(at 51.7652 166.37 0)
 			(effects
@@
 			)
 		)
-		(property "Footprint" ""
+		(property "Footprint" "Resistor_SMD:R_0805_2012Metric_Pad1.20x1.40mm_HandSolder"
 			(at 32.512 40.64 90)
 			(effects
@@
 			)
 		)
-		(property "Footprint" ""
+		(property "Footprint" "Capacitor_SMD:C_0805_2012Metric_Pad1.18x1.45mm_HandSolder"
 			(at 49.2252 31.75 0)
 			(effects
@@
 			)
 		)
-		(property "Footprint" ""
+		(property "Footprint" "Capacitor_SMD:C_0805_2012Metric_Pad1.18x1.45mm_HandSolder"
 			(at 51.7652 77.47 0)
 			(effects
@@
 			)
 		)
-		(property "Footprint" ""
+		(property "Footprint" "Capacitor_SMD:C_0805_2012Metric_Pad1.18x1.45mm_HandSolder"
 			(at 94.9452 31.75 0)
 			(effects
@@
 			)
 		)
-		(property "Footprint" ""
+		(property "Footprint" "Resistor_SMD:R_0805_2012Metric_Pad1.20x1.40mm_HandSolder"
 			(at 108.712 50.8 90)
 			(effects
@@
 			)
 		)
-		(property "Footprint" ""
+		(property "Footprint" "Capacitor_SMD:C_0805_2012Metric_Pad1.18x1.45mm_HandSolder"
 			(at 137.16 26.67 0)
 			(effects
@@
 			)
 		)
-		(property "Footprint" ""
+		(property "Footprint" "Capacitor_SMD:C_0805_2012Metric_Pad1.18x1.45mm_HandSolder"
 			(at 91.1352 123.19 0)
 			(effects
@@
 			)
 		)
-		(property "Footprint" ""
+		(property "Footprint" "Resistor_SMD:R_0805_2012Metric_Pad1.20x1.40mm_HandSolder"
 			(at 84.582 55.88 90)
 			(effects
@@
 			)
 		)
-		(property "Footprint" ""
+		(property "Footprint" "Capacitor_SMD:C_0805_2012Metric_Pad1.18x1.45mm_HandSolder"
 			(at 91.1352 78.74 0)
 			(effects
@@
 			)
 		)
-		(property "Footprint" ""
+		(property "Footprint" "Resistor_SMD:R_0805_2012Metric_Pad1.20x1.40mm_HandSolder"
 			(at 32.512 30.48 90)
 			(effects
@@
 			)
 		)
-		(property "Footprint" ""
+		(property "Footprint" "Capacitor_SMD:C_0805_2012Metric_Pad1.18x1.45mm_HandSolder"
 			(at 51.7652 121.92 0)
 			(effects
@@
 			)
 		)
-		(property "Footprint" ""
+		(property "Footprint" "Resistor_SMD:R_0805_2012Metric_Pad1.20x1.40mm_HandSolder"
 			(at 85.852 101.6 90)
 			(effects
@@
 			)
 		)
-		(property "Footprint" ""
+		(property "Footprint" "Capacitor_SMD:C_0805_2012Metric_Pad1.18x1.45mm_HandSolder"
 			(at 15.24 24.13 0)
 			(effects
@@
 			)
 		)
-		(property "Footprint" ""
+		(property "Footprint" "Resistor_SMD:R_0805_2012Metric_Pad1.20x1.40mm_HandSolder"
 			(at 85.852 146.05 90)
 			(effects
@@
 			)
 		)
-		(property "Footprint" ""
+		(property "Footprint" "Resistor_SMD:R_0805_2012Metric_Pad1.20x1.40mm_HandSolder"
 			(at 85.852 190.5 90)
 			(effects
@@
 			)
 		)
-		(property "Footprint" ""
+		(property "Footprint" "Capacitor_SMD:C_0805_2012Metric_Pad1.18x1.45mm_HandSolder"
 			(at 100.0252 58.42 0)
 			(effects
@@
 			)
 		)
-		(property "Footprint" ""
+		(property "Footprint" "Resistor_SMD:R_0805_2012Metric_Pad1.20x1.40mm_HandSolder"
 			(at 32.512 50.8 90)
 			(effects
@@
 			)
 		)
-		(property "Footprint" ""
+		(property "Footprint" "Capacitor_SMD:C_0805_2012Metric_Pad1.18x1.45mm_HandSolder"
 			(at 126.6952 31.75 0)
 			(effects
@@
 			)
 		)
-		(property "Footprint" ""
+		(property "Footprint" "Capacitor_SMD:C_0805_2012Metric_Pad1.18x1.45mm_HandSolder"
 			(at 91.1352 166.37 0)
 			(effects

Commit message: updates from Brian
Parts:
- removed C9: 0.1uF, Capacitor_SMD:C_0805_2012Metric_Pad1.18x1.45mm_HandSolder, symbol Device:C
- removed J1: Conn_01x02_Pin, Capacitor_SMD:C_0805_2012Metric_Pad1.18x1.45mm_HandSolder, symbol Connector:Conn_01x02_Pin
- added D1: SMCJ36CA, Footprints:SMCJ36CA, symbol SMCJ36CA:SMCJ36CA
- added D2, D3, D4, D5: LED, LED_SMD:LED_2512_6332Metric_Pad1.52x3.35mm_HandSolder, symbol Device:LED
- added Q1: CSD19537Q3, Footprints:TRANS_CSD19537Q3, symbol CSD19537Q3:CSD19537Q3
- added Q2: BSS138, Footprints:BSS138, symbol BSS138:BSS138
- added R4, R5, R6, R7: 29.4 kΩ, Resistor_SMD:R_0805_2012Metric_Pad1.20x1.40mm_HandSolder, symbol Device:R
- C1: value 0.1uF -> 1uF
- J1: renamed from J2; value Conn_01x02_Pin -> Conn_01x03_Pin; footprint Capacitor_SMD:C_0805_2012Metric_Pad1.18x1.45mm_HandSolder -> Connector_Wire:SolderWire-1.5sqmm_1x03_P7.8mm_D1.7mm_OD3.9mm; symbol Connector:Conn_01x02_Pin -> Connector:Conn_01x03_Pin
- U1, U2, U3, U7: footprint Package_DFN_QFN:Texas_RGE0024H_VQFN-24-1EP_4x4mm_P0.5mm_EP2.7x2.7mm_ThermalVias -> Footprints:QFN50P400X400X100-25N
- renumbered RILIM to RILIM4, RIMON to RIMON1
Connections:
- net GND: now also J1.3 (Pin_3), D1.1, D2.1 (K), D3.1 (K), D4.1 (K), D5.1 (K); no longer J1.2 (Pin_2)
- net at C13.1, C15.1, C16.1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: now also Q1.1, Q1.2, Q1.3; no longer C1.1, J1.1 (Pin_1), R1.1
- net at U7.16 (PGOOD): now also R4.1
- net at C10.1, C12.1, C14.1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: now also J1.1 (Pin_1)
- net at U7.3 (B_GATE): now also Q1.4, Q2.2
- net at U7.4 (DRV): now also Q2.1
- net at U7.5 (IN_SYS): now also C1.1, J1.2 (Pin_2), R1.1, U1.5 (IN_SYS), U2.5 (IN_SYS), U3.5 (IN_SYS), D1.2, Q1.5_8, Q2.3
- net at U3.15 (PGTH): now also R7.1
- net at U2.16 (PGOOD): now also R6.1
- net at U1.16 (PGOOD): now also R5.1
- new net: D2.2 (A), R4.2
- new net: D4.2 (A), R6.2
- new net: D3.2 (A), R5.2
- new net: D5.2 (A), R7.2

Commit message: pbc
Connections:
- net at R2.2, R3.1, U1.7 (OVP)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: no longer U3.7 (OVP)
Changed lines of the file:
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@@
-	)
-	(junction
-		(at 41.91 135.89)
-		(diameter 0)
-		(color 0 0 0 0)
 	)
 	(junction
@@
 	(wire
 		(pts
-			(xy 41.91 180.34) (xy 59.69 180.34)
-		)
-		(stroke
-			(width 0)
-			(type default)
-		)
-	)
-	(wire
-		(pts
 			(xy 87.63 194.31) (xy 72.39 194.31)
 		)
@@
 	(wire
 		(pts
-			(xy 41.91 135.89) (xy 41.91 180.34)
-		)
-		(stroke
+			(xy -2.54 180.34) (xy 59.69 180.34)
+		)
+		(stroke
