File: EFUSE2024/EFUSE2024.kicad_sch (KiCad schematic)
At the start: 34 parts, among them J1 Conn_01x03_Pin, Q1 CSD19537Q3, Q2 BSS138, U1 TPS26630RGE, U2 TPS26630RGE, U3 TPS26630RGE, U7 TPS26630RGE

Commit message: fixed up PCB
Parts:
- removed C12, C13, C14, C16, C17, C18: 0.1uF, Capacitor_SMD:C_0805_2012Metric_Pad1.18x1.45mm_HandSolder, symbol Device:C
Connections:
- net at C15.1, Q1.1, Q1.2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: now also Q2.1, U1.4 (DRV), U2.4 (DRV), U3.4 (DRV), U7.4 (DRV)
- net at Q1.4, Q2.2, U7.3 (B_GATE): now also U1.3 (B_GATE), U2.3 (B_GATE), U3.3 (B_GATE)
- net at R2.2, R3.1, U1.7 (OVP)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: now also U3.7 (OVP)
- net at U3.15 (PGTH): no longer R7.1
- net at U3.16 (PGOOD): now also R7.1
Other:
- moved on the sheet: C15

Commit message: updates
Connections:
- net at C15.1, Q1.1, Q1.2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: no longer Q2.1, U1.4 (DRV), U2.4 (DRV), U3.4 (DRV), U7.4 (DRV)
- new net: Q2.1, U1.4 (DRV), U2.4 (DRV), U3.4 (DRV), U7.4 (DRV)
Changed lines of the file:
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@@
 	)
 	(junction
+		(at 52.07 34.29)
+		(diameter 0)
+		(color 0 0 0 0)
+	)
+	(junction
 		(at 93.98 133.35)
 		(diameter 0)
@@
 	)
 	(junction
-		(at 93.98 43.18)
-		(diameter 0)
-		(color 0 0 0 0)
-	)
-	(junction
 		(at 45.72 39.37)
 		(diameter 0)
@@
 	)
 	(junction
-		(at 90.17 69.85)
-		(diameter 0)
-		(color 0 0 0 0)
-	)
-	(junction
 		(at 93.98 88.9)
 		(diameter 0)
@@
 	)
 	(junction
-		(at 50.8 34.29)
-		(diameter 0)
-		(color 0 0 0 0)
-	)
-	(junction
 		(at 99.06 48.26)
 		(diameter 0)
@@
 	)
 	(junction
-		(at 90.17 114.3)
-		(diameter 0)
-		(color 0 0 0 0)
-	)
-	(junction
 		(at 102.87 138.43)
 		(diameter 0)
@@
 	)
 	(junction
-		(at 110.49 45.72)
-		(diameter 0)
-		(color 0 0 0 0)
-	)
-	(junction
 		(at 53.34 74.93)
 		(diameter 0)
@@
 	)
 	(junction
-		(at 50.8 69.85)
-		(diameter 0)
-		(color 0 0 0 0)
-	)
-	(junction
 		(at 106.68 135.89)
 		(diameter 0)
@@
 	(wire
 		(pts
-			(xy 50.8 80.01) (xy 50.8 69.85)
-		)
-		(stroke
-			(width 0)
-			(type default)
-		)
-	)
-	(wire
-		(pts
 			(xy 85.09 97.79) (xy 87.63 97.79)
 		)
@@
 	(wire
 		(pts
-			(xy 52.07 80.01) (xy 50.8 80.01)
-		)
-		(stroke
-			(width 0)
-			(type default)
-		)
-	)
-	(wire
-		(pts
-			(xy 90.17 114.3) (xy 90.17 115.57)
-		)
-		(stroke
-			(width 0)
-			(type default)
-		)
-	)
-	(wire
-		(pts
 			(xy 110.49 45.72) (xy 110.49 46.99)
 		)
@@
 	(wire
 		(pts
+			(xy 45.72 39.37) (xy 45.72 85.09)
+		)
+		(stroke
+			(width 0)
+			(type default)
+		)
+	)
+	(wire
+		(pts
 			(xy 99.06 48.26) (xy 102.87 48.26)
 		)
@@
 	(wire
 		(pts
-			(xy 50.8 34.29) (xy 48.26 34.29)
+			(xy 48.26 34.29) (xy 52.07 34.29)
 		)
 		(stroke
@@
 	(wire
 		(pts
-			(xy 85.09 114.3) (xy 90.17 114.3)
+			(xy 85.09 114.3) (xy 119.38 114.3)
 		)
 		(stroke
@@
 	(wire
 		(pts
-			(xy 90.17 69.85) (xy 90.17 71.12)
-		)
-		(stroke
-			(width 0)
-			(type default)
-		)
-	)
-	(wire
-		(pts
 			(xy 45.72 129.54) (xy 45.72 173.99)
 		)
@@
 	(wire
 		(pts
-			(xy 50.8 69.85) (xy 50.8 34.29)
+			(xy 52.07 34.29) (xy 52.07 80.01)
 		)
 		(stroke
@@
 	(wire
 		(pts
-			(xy 90.17 69.85) (xy 119.38 69.85)
-		)
-		(stroke
-			(width 0)
-			(type default)
-		)
-	)
-	(wire
-		(pts
 			(xy 50.8 24.13) (xy 54.61 24.13)
 		)
@@
 	(wire
 		(pts
-			(xy 90.17 114.3) (xy 119.38 114.3)
-		)
-		(stroke
-			(width 0)
-			(type default)
-		)
-	)
-	(wire
-		(pts
 			(xy 41.91 91.44) (xy 59.69 91.44)
 		)
@@
 	(wire
 		(pts
-			(xy 50.8 69.85) (xy 54.61 69.85)
-		)
-		(stroke
-			(width 0)
-			(type default)
-		)
-	)
-	(wire
-		(pts
 			(xy 72.39 149.86) (xy 59.69 149.86)
 		)
@@
 	(wire
 		(pts
-			(xy 93.98 43.18) (xy 100.33 43.18)
-		)
-		(stroke
-			(width 0)
-			(type default)
-		)
-	)
-	(wire
-		(pts
 			(xy 72.39 147.32) (xy 72.39 149.86)
 		)
@@
 	(wire
 		(pts
-			(xy 59.69 34.29) (xy 50.8 34.29)
+			(xy 59.69 34.29) (xy 52.07 34.29)
 		)
 		(stroke
@@
 	(wire
 		(pts
-			(xy 45.72 39.37) (xy 45.72 85.09)
-		)
-		(stroke
-			(width 0)
-			(type default)
-		)
-	)
-	(wire
-		(pts
 			(xy 148.59 54.61) (xy 148.59 60.96)
 		)
@@
 	(wire
 		(pts
-			(xy 85.09 69.85) (xy 90.17 69.85)
+			(xy 85.09 69.85) (xy 119.38 69.85)
 		)
 		(stroke
@@
 	(wire
 		(pts
-			(xy 110.49 45.72) (xy 113.03 45.72)
-		)
-		(stroke
-			(width 0)
-			(type default)
-		)
-	)
-	(wire
-		(pts
 			(xy 52.07 124.46) (xy 52.07 168.91)
 		)
@@
 		(on_board yes)
 		(dnp no)
-		(fields_autoplaced yes)
 		(property "Reference" "#PWR017"
 			(at 72.39 66.04 0)
@@
 		)
 		(property "Value" "GND"
-			(at 72.39 64.77 0)
+			(at 75.946 61.976 0)
 			(effects
 				(font

Commit message: adding gerber files
Parts:
- renumbered C11 to C1, C1 to C2, C10 to C3, C15 to C4, D5 to D3, D3 to D4, D4 to D5, R7 to R5, R5 to R7, RILIM4 to RILIM1, RILIM1 to RILIM2, RILIM2 to RILIM3, RILIM3 to RILIM4, U7 to U1, U1 to U2, U2 to U3, U3 to U4
Changed lines of the file:
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@@
 		(on_board yes)
 		(dnp no)
-		(property "Reference" "C1"
+		(property "Reference" "C2"
 			(at 27.686 26.924 0)
 			(effects
@@
 			(project ""
 				(path "/c5be8a64-8a8b-4055-8c54-4d0f5ad85ba2"
-					(reference "C1")
+					(reference "C2")
 					(unit 1)
 				)
@@
 		(dnp no)
 		(fields_autoplaced yes)
-		(property "Reference" "U7"
+		(property "Reference" "U1"
 			(at 74.5841 16.51 0)
 			(effects
@@
 			(project ""
 				(path "/c5be8a64-8a8b-4055-8c54-4d0f5ad85ba2"
-					(reference "U7")
+					(reference "U1")
 					(unit 1)
 				)
@@
 		(on_board yes)
 		(dnp no)
-		(property "Reference" "U3"
+		(property "Reference" "U4"
 			(at 66.294 154.686 0)
 			(effects
@@
 			(project "EFUSE2024"
 				(path "/c5be8a64-8a8b-4055-8c54-4d0f5ad85ba2"
-					(reference "U3")
+					(reference "U4")
 					(unit 1)
 				)
@@
 		(dnp no)
 		(fields_autoplaced yes)
-		(property "Reference" "D4"
+		(property "Reference" "D5"
 			(at 154.94 145.0974 90)
 			(effects
@@
 			(project ""
 				(path "/c5be8a64-8a8b-4055-8c54-4d0f5ad85ba2"
-					(reference "D4")
+					(reference "D5")
 					(unit 1)
 				)
@@
 		(on_board yes)
 		(dnp no)
-		(property "Reference" "C10"
+		(property "Reference" "C3"
 			(at 97.79 26.6699 0)
 			(effects
@@
 			(project "EFUSE2024"
 				(path "/c5be8a64-8a8b-4055-8c54-4d0f5ad85ba2"
-					(reference "C10")
+					(reference "C3")
 					(unit 1)
 				)
@@
 		(dnp no)
 		(fields_autoplaced yes)
-		(property "Reference" "D3"
+		(property "Reference" "D4"
 			(at 154.94 98.1074 90)
 			(effects
@@
 			(project ""
 				(path "/c5be8a64-8a8b-4055-8c54-4d0f5ad85ba2"
-					(reference "D3")
+					(reference "D4")
 					(unit 1)
 				)
@@
 		(on_board yes)
 		(dnp no)
-		(property "Reference" "RILIM4"
+		(property "Reference" "RILIM1"
 			(at 87.376 54.61 0)
 			(effects
@@
 			(project "EFUSE2024"
 				(path "/c5be8a64-8a8b-4055-8c54-4d0f5ad85ba2"
-					(reference "RILIM4")
+					(reference "RILIM1")
 					(unit 1)
 				)
@@
 		(on_board yes)
 		(dnp no)
-		(property "Reference" "C15"
+		(property "Reference" "C4"
 			(at 14.732 120.65 0)
 			(effects
@@
 			(project "EFUSE2024"
 				(path "/c5be8a64-8a8b-4055-8c54-4d0f5ad85ba2"
-					(reference "C15")
+					(reference "C4")
 					(unit 1)
 				)
@@
 		(on_board yes)
 		(dnp no)
-		(property "Reference" "RILIM1"
+		(property "Reference" "RILIM2"
 			(at 88.646 100.33 0)
 			(effects
@@
 			(project "EFUSE2024"
 				(path "/c5be8a64-8a8b-4055-8c54-4d0f5ad85ba2"
-					(reference "RILIM1")
+					(reference "RILIM2")
 					(unit 1)
 				)
@@
 		(on_board yes)
 		(dnp no)
-		(property "Reference" "U2"
+		(property "Reference" "U3"
 			(at 67.564 110.236 0)
 			(effects
@@
 			(project "EFUSE2024"
 				(path "/c5be8a64-8a8b-4055-8c54-4d0f5ad85ba2"
-					(reference "U2")
+					(reference "U3")
 					(unit 1)
 				)
@@
 		(dnp no)
 		(fields_autoplaced yes)
-		(property "Reference" "D5"
+		(property "Reference" "D3"
 			(at 143.51 179.3874 90)
 			(effects
@@
 			(project "EFUSE2024"
 				(path "/c5be8a64-8a8b-4055-8c54-4d0f5ad85ba2"
-					(reference "D5")
+					(reference "D3")
 					(unit 1)
 				)
@@
 		(on_board yes)
 		(dnp no)
-		(property "Reference" "RILIM2"
+		(property "Reference" "RILIM3"
 			(at 88.646 144.78 0)
 			(effects
@@
 			(project "EFUSE2024"
 				(path "/c5be8a64-8a8b-4055-8c54-4d0f5ad85ba2"
-					(reference "RILIM2")
+					(reference "RILIM3")
 					(unit 1)
 				)
@@
 		(on_board yes)
 		(dnp no)
-		(property "Reference" "U1"
+		(property "Reference" "U2"
 			(at 67.056 65.786 0)
 			(effects
@@
 			(project "EFUSE2024"
 				(path "/c5be8a64-8a8b-4055-8c54-4d0f5ad85ba2"
-					(reference "U1")
+					(reference "U2")
 					(unit 1)
 				)
@@
 		(on_board yes)
 		(dnp no)
-		(property "Reference" "R5"
+		(property "Reference" "R7"
 			(at 153.162 84.836 0)
 			(effects
@@
 			(project "EFUSE2024"
 				(path "/c5be8a64-8a8b-4055-8c54-4d0f5ad85ba2"
-					(reference "R5")
+					(reference "R7")
 					(unit 1)
 				)
@@
 		(on_board yes)
 		(dnp no)
-		(property "Reference" "RILIM3"
+		(property "Reference" "RILIM4"
 			(at 88.646 189.23 0)
 			(effects
@@
 			(project "EFUSE2024"
 				(path "/c5be8a64-8a8b-4055-8c54-4d0f5ad85ba2"
-					(reference "RILIM3")
+					(reference "RILIM4")
 					(unit 1)
 				)
@@
 		(on_board yes)
 		(dnp no)
-		(property "Reference" "C11"
+		(property "Reference" "C1"
 			(at 94.742 57.404 0)
 			(effects
@@
 			(project "EFUSE2024"
 				(path "/c5be8a64-8a8b-4055-8c54-4d0f5ad85ba2"
-					(reference "C11")
+					(reference "C1")
 					(unit 1)
 				)
@@
 		(on_board yes)
 		(dnp no)
-		(property "Reference" "R7"
+		(property "Reference" "R5"
 			(at 141.732 163.576 0)
 			(effects
@@
 			(project "EFUSE2024"
 				(path "/c5be8a64-8a8b-4055-8c54-4d0f5ad85ba2"
-					(reference "R7")
-					(unit 1)
-				)
+					(reference "R5")
+					(unit 1)
+				)

Commit message: final update
Parts:
- added JP1, JP2, JP3, JP4: Jumper_2_Bridged, Jumper:SolderJumper-2_P1.3mm_Bridged2Bar_Pad1.0x1.5mm, symbol Jumper:Jumper_2_Bridged
- D1: value SMCJ36CA -> DIOM6859X262N
- Q2: value BSS138 -> SOT95P240X111-3N
- renumbered C2 to C1, C3 to C10, C1 to C11, C4 to C15
Connections:
- net GND: now also JP1.1 (A), JP2.1 (A), JP3.1 (A), JP4.1 (A); no longer U1.11 (MODE), U2.11 (MODE), U3.11 (MODE), U4.11 (MODE)
- net at C15.1, Q1.1, Q1.2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: now also Q2.1, U1.4 (DRV), U2.4 (DRV), U3.4 (DRV), U4.4 (DRV)
- new net: JP4.2 (B), U1.11 (MODE)
- new net: JP2.2 (B), U4.11 (MODE)
- new net: JP3.2 (B), U2.11 (MODE)
- new net: JP1.2 (B), U3.11 (MODE)
