File: EFUSE2024/EFUSE2024.kicad_pcb (KiCad board)
At the start: 2 copper layers, 34 parts, among them J1 Conn_01x03_Pin, Q1 CSD19537Q3, Q2 SOT95P240X111-3N, U1 TPS26630RGE, U2 TPS26630RGE, U3 TPS26630RGE, U7 TPS26630RGE

Commit message: PBC changes
Parts:
- D1: value DIOM6859X262N -> SMCJ36CA
- Q2: value SOT95P240X111-3N -> BSS138
- moved C18 56.9 mm to (137.3, 28.6)
- moved C11 52.7 mm to (133.5, 28.8)
- moved Q1 47.1 mm to (111.5, 29.7), turned to 180 degrees
- moved J1 43.4 mm to (112.9, 16.4)
- moved RIMON1 43.0 mm to (138.9, 47.4)
- moved RILIM3 42.1 mm to (137.0, 41.4), turned to 90 degrees
- moved C10 41.7 mm to (126.2, 34.0)
- moved RILIM4 40.0 mm to (126.5, 41.7), turned to 90 degrees
- moved Q2 38.9 mm to (105.5, 31.4)
- moved RILIM1 38.6 mm to (139.2, 41.4), turned to -90 degrees
- moved RILIM2 38.2 mm to (134.2, 41.2), turned to 90 degrees
- moved C1 33.4 mm to (100.9, 28.8)
- moved D1 29.8 mm to (93.4, 28.3), turned to -90 degrees
- moved U1 28.8 mm to (118.9, 36.8)
- moved R1 26.6 mm to (107.4, 36.4)
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
Commit message: pbc
Parts:
- moved U7 43.2 mm to (116.9, 40.2)
- moved U1 15.4 mm to (116.6, 52.0)
- moved U2 15.2 mm to (116.5, 62.1)
- moved U3 7.96 mm to (116.1, 73.2)
- moved Q1 6.17 mm to (107.5, 25.0)
- moved R1 5.50 mm to (101.9, 36.4)
- moved R2 5.50 mm to (101.8, 40.7)
- moved R3 5.50 mm to (101.5, 44.6)
- moved RILIM1 5.30 mm to (144.5, 41.4)
- moved RILIM2 3.71 mm to (130.5, 41.5)
- moved Q2 3.58 mm to (107.1, 34.5)
- moved RILIM4 2.69 mm to (124.5, 43.5)
Changed lines of the file:
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@@
 	(footprint "Resistor_SMD:R_0805_2012Metric_Pad1.20x1.40mm_HandSolder"
 		(layer "F.Cu")
-		(at 107.3 40.7)
+		(at 101.8 40.7)
 		(descr "Resistor SMD 0805 (2012 Metric), square (rectangular) end terminal, IPC_7351 nominal with elongated pad for handsoldering. (Body size source: IPC-SM-782 page 72, https://www.pcb-3d.com/wordpress/wp-content/uploads/ipc-sm-782a_amendment_1_and_2.pdf), generated with kicad-footprint-generator")
 		(tags "resistor handsolder")
@@
 	(footprint "Resistor_SMD:R_0805_2012Metric_Pad1.20x1.40mm_HandSolder"
 		(layer "F.Cu")
-		(at 126.5 41.7 90)
+		(at 124.5 43.5 90)
 		(descr "Resistor SMD 0805 (2012 Metric), square (rectangular) end terminal, IPC_7351 nominal with elongated pad for handsoldering. (Body size source: IPC-SM-782 page 72, https://www.pcb-3d.com/wordpress/wp-content/uploads/ipc-sm-782a_amendment_1_and_2.pdf), generated with kicad-footprint-generator")
 		(tags "resistor handsolder")
@@
 	(footprint "Footprints:TRANS_CSD19537Q3"
 		(layer "F.Cu")
-		(at 111.5 29.7 180)
+		(at 107.5 25 180)
 		(property "Reference" "Q1"
-			(at 0.54 -2.508 360)
+			(at 0.54 -2.508 0)
 			(layer "F.SilkS")
 			(effects
@@
 		)
 		(property "Value" "CSD19537Q3"
-			(at 6.128 2.508 360)
+			(at 6.128 2.508 0)
 			(layer "F.Fab")
 			(effects
@@
 		)
 		(property "Footprint" "Footprints:TRANS_CSD19537Q3"
-			(at 0 0 360)
+			(at 0 0 0)
 			(layer "F.Fab")
 			(hide yes)
@@
 		)
 		(property "Datasheet" ""
-			(at 0 0 360)
+			(at 0 0 0)
 			(layer "F.Fab")
 			(hide yes)
@@
 		)
 		(property "Description" ""
-			(at 0 0 360)
+			(at 0 0 0)
 			(layer "F.Fab")
 			(hide yes)
@@
 	(footprint "Footprints:QFN50P400X400X100-25N"
 		(layer "F.Cu")
-		(at 108.75 82.6575)
+		(at 116.9125 40.25)
 		(property "Reference" "U7"
-			(at 0.175 -3.635 0)
+			(at 0.175 -3.635 360)
 			(layer "F.SilkS")
 			(effects
@@
 		)
 		(property "Value" "TPS26630RGE"
-			(at 10.335 3.635 0)
+			(at 10.335 3.635 360)
 			(layer "F.Fab")
 			(effects
@@
 		)
 		(property "Footprint" "Footprints:QFN50P400X400X100-25N"
-			(at 0 0 0)
+			(at 0 0 360)
 			(layer "F.Fab")
 			(hide yes)
@@
 		)
 		(property "Datasheet" "https://www.ti.com/lit/ds/symlink/tps2663.pdf"
-			(at 0 0 0)
+			(at 0 0 360)
 			(layer "F.Fab")
 			(hide yes)
@@
 		)
 		(property "Description" "60V, 6A Power Limiting, Surge Protection Industrial eFuse, Adjustable Overvoltage cut-off, Active Current Limiting, VQFN-24"
-			(at 0 0 0)
+			(at 0 0 360)
 			(layer "F.Fab")
 			(hide yes)
@@
 	(footprint "Resistor_SMD:R_0805_2012Metric_Pad1.20x1.40mm_HandSolder"
 		(layer "F.Cu")
-		(at 139.2 41.4 -90)
+		(at 144.5 41.4 -90)
 		(descr "Resistor SMD 0805 (2012 Metric), square (rectangular) end terminal, IPC_7351 nominal with elongated pad for handsoldering. (Body size source: IPC-SM-782 page 72, https://www.pcb-3d.com/wordpress/wp-content/uploads/ipc-sm-782a_amendment_1_and_2.pdf), generated with kicad-footprint-generator")
 		(tags "resistor handsolder")
@@
 	(footprint "Footprints:QFN50P400X400X100-25N"
 		(layer "F.Cu")
-		(at 118.81375 47.1)
+		(at 116.5 62.1)
 		(property "Reference" "U2"
 			(at 0.175 -3.635 0)
@@
 	(footprint "Footprints:QFN50P400X400X100-25N"
 		(layer "F.Cu")
-		(at 108.75 76.3475)
+		(at 116.0875 73.25)
 		(property "Reference" "U3"
 			(at 0.175 -3.635 0)
@@
 	(footprint "Resistor_SMD:R_0805_2012Metric_Pad1.20x1.40mm_HandSolder"
 		(layer "F.Cu")
-		(at 134.2 41.2 90)
+		(at 130.5 41.5 90)
 		(descr "Resistor SMD 0805 (2012 Metric), square (rectangular) end terminal, IPC_7351 nominal with elongated pad for handsoldering. (Body size source: IPC-SM-782 page 72, https://www.pcb-3d.com/wordpress/wp-content/uploads/ipc-sm-782a_amendment_1_and_2.pdf), generated with kicad-footprint-generator")
 		(tags "resistor handsolder")
 		(property "Reference" "RILIM2"
-			(at 0 -1.65 90)
+			(at 0 0 90)
 			(layer "F.SilkS")
 			(effects
@@
 	(footprint "Footprints:QFN50P400X400X100-25N"
 		(layer "F.Cu")
-		(at 118.9 36.8)
+		(at 116.6 52)
 		(property "Reference" "U1"
 			(at 0.175 -3.635 0)
@@
 	(footprint "Resistor_SMD:R_0805_2012Metric_Pad1.20x1.40mm_HandSolder"
 		(layer "F.Cu")
-		(at 107.4 36.4)
+		(at 101.9 36.4)
 		(descr "Resistor SMD 0805 (2012 Metric), square (rectangular) end terminal, IPC_7351 nominal with elongated pad for handsoldering. (Body size source: IPC-SM-782 page 72, https://www.pcb-3d.com/wordpress/wp-content/uploads/ipc-sm-782a_amendment_1_and_2.pdf), generated with kicad-footprint-generator")
 		(tags "resistor handsolder")
@@
 	(footprint "Resistor_SMD:R_0805_2012Metric_Pad1.20x1.40mm_HandSolder"
 		(layer "F.Cu")
-		(at 107 44.6)
+		(at 101.5 44.6)
 		(descr "Resistor SMD 0805 (2012 Metric), square (rectangular) end terminal, IPC_7351 nominal with elongated pad for handsoldering. (Body size source: IPC-SM-782 page 72, https://www.pcb-3d.com/wordpress/wp-content/uploads/ipc-sm-782a_amendment_1_and_2.pdf), generated with kicad-footprint-generator")
 		(tags "resistor handsolder")
@@
 	(footprint "Footprints:BSS138"
 		(layer "F.Cu")
-		(at 105.46 31.35)
+		(at 107.06 34.55)
 		(property "Reference" "Q2"
 			(at 0.032 -2.4064 0)

Commit message: PBC
Parts:
- moved C12 43.2 mm to (127.5, 37.0)
- moved RILIM3 41.4 mm to (122.0, 80.0)
- moved D2 41.2 mm to (144.0, 27.0)
- moved C13 40.6 mm to (115.0, 39.0)
- moved R4 35.5 mm to (136.5, 27.0)
- moved D3 33.7 mm to (144.5, 40.5)
- moved C17 32.1 mm to (122.0, 73.5)
- moved RILIM2 28.2 mm to (122.5, 68.5)
- moved R5 25.7 mm to (136.0, 40.0)
- moved C14 23.5 mm to (122.5, 60.0)
- moved Q1 19.5 mm to (124.6, 15.5), turned to 0 degrees
- moved Q2 18.5 mm to (110.9, 16.4), turned to 180 degrees
- moved R2 17.0 mm to (115.0, 30.0), turned to 180 degrees
- moved R1 16.7 mm to (115.0, 26.0)
- moved R3 16.7 mm to (114.0, 33.5)
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
Commit message: PCB
Parts:
- moved RILIM2 26.5 mm to (123.5, 42.0)
- moved D4 24.7 mm to (133.5, 41.0)
- moved R6 24.5 mm to (128.0, 38.0)
- moved C15 23.9 mm to (109.5, 37.5), turned to 180 degrees
- moved C14 23.0 mm to (123.5, 37.0), turned to -90 degrees
- moved U2 22.2 mm to (118.4, 40.0)
- moved RILIM3 22.0 mm to (115.5, 59.0), turned to 0 degrees
- moved D5 20.7 mm to (133.5, 56.5)
- moved U3 20.2 mm to (110.2, 53.9)
- moved C17 19.9 mm to (118.0, 54.0), turned to -90 degrees
- moved R7 18.6 mm to (128.1, 55.0)
- moved C18 18.5 mm to (128.5, 16.5), turned to -90 degrees
- moved C16 15.8 mm to (102.0, 55.0), turned to 180 degrees
- moved D3 13.6 mm to (133.5, 32.5), turned to 90 degrees
- moved R5 13.2 mm to (128.0, 29.5)
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
Commit message: PCB
Parts:
- moved Q2 69.8 mm to (100.9, 85.5)
- moved D2 67.1 mm to (129.5, 85.0)
- moved C15 66.9 mm to (95.6, 103.0), turned to -90 degrees
- moved R5 66.6 mm to (124.0, 96.0)
- moved Q1 65.5 mm to (101.0, 81.0)
- moved C10 65.4 mm to (112.5, 81.0)
- moved C18 65.4 mm to (117.5, 81.0)
- moved C13 65.3 mm to (95.6, 93.3), turned to -90 degrees
- moved RILIM4 65.1 mm to (112.3, 86.1)
- moved R3 64.9 mm to (96.0, 89.5)
- moved C12 64.8 mm to (112.6, 90.9)
- moved U7 64.6 mm to (107.0, 84.1)
- moved U2 64.5 mm to (107.0, 103.5)
- moved C14 64.4 mm to (112.6, 100.5)
- moved RILIM2 64.4 mm to (112.6, 105.5)
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
Commit message: pbc
Parts:
- moved C10 3.00 mm to (115.5, 81.0)
- moved C11 3.00 mm to (119.5, 86.0)
- moved C18 3.00 mm to (120.5, 81.0)
- moved RILIM4 3.00 mm to (115.3, 86.1)
- moved RIMON1 3.00 mm to (124.0, 86.0)
- moved RILIM3 2.60 mm to (115.5, 117.0)
- moved C12 2.40 mm to (115.0, 90.9)
- moved C14 2.40 mm to (115.0, 100.5)
- moved C17 2.40 mm to (115.0, 111.5)
- moved RILIM1 2.40 mm to (115.0, 95.5)
- moved RILIM2 2.40 mm to (115.0, 105.5)
- moved U1 1.61 mm to (108.7, 93.2)
- moved U2 1.61 mm to (108.6, 103.8)
- moved U3 1.61 mm to (108.6, 114.2)
- moved U7 1.61 mm to (108.6, 84.3)
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Changed lines of the file:
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@@
 	(footprint "Capacitor_SMD:C_0805_2012Metric_Pad1.18x1.45mm_HandSolder"
 		(layer "F.Cu")
-		(at 117.5 81 -90)
+		(at 120.5 81 -90)
 		(descr "Capacitor SMD 0805 (2012 Metric), square (rectangular) end terminal, IPC_7351 nominal with elongated pad for handsoldering. (Body size source: IPC-SM-782 page 76, https://www.pcb-3d.com/wordpress/wp-content/uploads/ipc-sm-782a_amendment_1_and_2.pdf, https://docs.google.com/spreadsheets/d/1BsfQQcO9C6DZCsRaXUlFlo91Tg2WpOkGARC1WS5S8t0/edit?usp=sharing), generated with kicad-footprint-generator")
 		(tags "capacitor handsolder")
@@
 	(footprint "Capacitor_SMD:C_0805_2012Metric_Pad1.18x1.45mm_HandSolder"
 		(layer "F.Cu")
-		(at 112.6 90.8875 -90)
+		(at 115 90.9 -90)
 		(descr "Capacitor SMD 0805 (2012 Metric), square (rectangular) end terminal, IPC_7351 nominal with elongated pad for handsoldering. (Body size source: IPC-SM-782 page 76, https://www.pcb-3d.com/wordpress/wp-content/uploads/ipc-sm-782a_amendment_1_and_2.pdf, https://docs.google.com/spreadsheets/d/1BsfQQcO9C6DZCsRaXUlFlo91Tg2WpOkGARC1WS5S8t0/edit?usp=sharing), generated with kicad-footprint-generator")
 		(tags "capacitor handsolder")
@@
 		)
 		(fp_text user "${REFERENCE}"
-			(at 4.5 7.5 90)
+			(at 4.7625 5.9125 90)
 			(layer "F.Fab")
 			(effects
@@
 	(footprint "Capacitor_SMD:C_0805_2012Metric_Pad1.18x1.45mm_HandSolder"
 		(layer "F.Cu")
-		(at 112.6 100.5 -90)
+		(at 115 100.5125 -90)
 		(descr "Capacitor SMD 0805 (2012 Metric), square (rectangular) end terminal, IPC_7351 nominal with elongated pad for handsoldering. (Body size source: IPC-SM-782 page 76, https://www.pcb-3d.com/wordpress/wp-content/uploads/ipc-sm-782a_amendment_1_and_2.pdf, https://docs.google.com/spreadsheets/d/1BsfQQcO9C6DZCsRaXUlFlo91Tg2WpOkGARC1WS5S8t0/edit?usp=sharing), generated with kicad-footprint-generator")
 		(tags "capacitor handsolder")
@@
 	(footprint "Resistor_SMD:R_0805_2012Metric_Pad1.20x1.40mm_HandSolder"
 		(layer "F.Cu")
-		(at 112.35 86.0875 -90)
+		(at 115.35 86.0875 -90)
 		(descr "Resistor SMD 0805 (2012 Metric), square (rectangular) end terminal, IPC_7351 nominal with elongated pad for handsoldering. (Body size source: IPC-SM-782 page 72, https://www.pcb-3d.com/wordpress/wp-content/uploads/ipc-sm-782a_amendment_1_and_2.pdf), generated with kicad-footprint-generator")
 		(tags "resistor handsolder")
@@
 	(footprint "Footprints:TRANS_CSD19537Q3"
 		(layer "F.Cu")
-		(at 101 80.9875)
+		(at 102 80.5)
 		(property "Reference" "Q1"
 			(at 0.54 -2.508 0)
@@
 	(footprint "Resistor_SMD:R_0805_2012Metric_Pad1.20x1.40mm_HandSolder"
 		(layer "F.Cu")
-		(at 121 86 -90)
+		(at 124 86 -90)
 		(descr "Resistor SMD 0805 (2012 Metric), square (rectangular) end terminal, IPC_7351 nominal with elongated pad for handsoldering. (Body size source: IPC-SM-782 page 72, https://www.pcb-3d.com/wordpress/wp-content/uploads/ipc-sm-782a_amendment_1_and_2.pdf), generated with kicad-footprint-generator")
 		(tags "resistor handsolder")
@@
 	(footprint "Capacitor_SMD:C_0805_2012Metric_Pad1.18x1.45mm_HandSolder"
 		(layer "F.Cu")
-		(at 116.5 86 -90)
+		(at 119.5 86 -90)
 		(descr "Capacitor SMD 0805 (2012 Metric), square (rectangular) end terminal, IPC_7351 nominal with elongated pad for handsoldering. (Body size source: IPC-SM-782 page 76, https://www.pcb-3d.com/wordpress/wp-content/uploads/ipc-sm-782a_amendment_1_and_2.pdf, https://docs.google.com/spreadsheets/d/1BsfQQcO9C6DZCsRaXUlFlo91Tg2WpOkGARC1WS5S8t0/edit?usp=sharing), generated with kicad-footprint-generator")
 		(tags "capacitor handsolder")
@@
 	(footprint "Footprints:QFN50P400X400X100-25N"
 		(layer "F.Cu")
-		(at 107 84.075)
+		(at 108.5875 84.3375)
 		(property "Reference" "U7"
 			(at 0.175 -3.635 0)
@@
 		)
 		(property "Value" "TPS26630RGE"
-			(at 10.335 3.635 0)
+			(at 13.335 3.635 0)
 			(layer "F.Fab")
 			(effects
@@
 	(footprint "Resistor_SMD:R_0805_2012Metric_Pad1.20x1.40mm_HandSolder"
 		(layer "F.Cu")
-		(at 113.1 117.9875)
+		(at 115.5 117)
 		(descr "Resistor SMD 0805 (2012 Metric), square (rectangular) end terminal, IPC_7351 nominal with elongated pad for handsoldering. (Body size source: IPC-SM-782 page 72, https://www.pcb-3d.com/wordpress/wp-content/uploads/ipc-sm-782a_amendment_1_and_2.pdf), generated with kicad-footprint-generator")
 		(tags "resistor handsolder")
@@
 	(footprint "Resistor_SMD:R_0805_2012Metric_Pad1.20x1.40mm_HandSolder"
 		(layer "F.Cu")
-		(at 112.6 95.4875 -90)
+		(at 115 95.5 -90)
 		(descr "Resistor SMD 0805 (2012 Metric), square (rectangular) end terminal, IPC_7351 nominal with elongated pad for handsoldering. (Body size source: IPC-SM-782 page 72, https://www.pcb-3d.com/wordpress/wp-content/uploads/ipc-sm-782a_amendment_1_and_2.pdf), generated with kicad-footprint-generator")
 		(tags "resistor handsolder")
@@
 	(footprint "Footprints:QFN50P400X400X100-25N"
 		(layer "F.Cu")
-		(at 107 103.5)
+		(at 108.5875 103.7625)
 		(property "Reference" "U2"
 			(at 0.175 -3.635 0)
@@
 	(footprint "Footprints:QFN50P400X400X100-25N"
 		(layer "F.Cu")
-		(at 107 113.9875)
+		(at 108.5875 114.25)
 		(property "Reference" "U3"
 			(at 0.175 -3.635 0)
@@
 	(footprint "Capacitor_SMD:C_0805_2012Metric_Pad1.18x1.45mm_HandSolder"
 		(layer "F.Cu")
-		(at 112.6 111.525 -90)
+		(at 115 111.5375 -90)
 		(descr "Capacitor SMD 0805 (2012 Metric), square (rectangular) end terminal, IPC_7351 nominal with elongated pad for handsoldering. (Body size source: IPC-SM-782 page 76, https://www.pcb-3d.com/wordpress/wp-content/uploads/ipc-sm-782a_amendment_1_and_2.pdf, https://docs.google.com/spreadsheets/d/1BsfQQcO9C6DZCsRaXUlFlo91Tg2WpOkGARC1WS5S8t0/edit?usp=sharing), generated with kicad-footprint-generator")
 		(tags "capacitor handsolder")
@@
 	(footprint "Resistor_SMD:R_0805_2012Metric_Pad1.20x1.40mm_HandSolder"
 		(layer "F.Cu")
-		(at 112.6 105.4875 90)
+		(at 115 105.5 90)
 		(descr "Resistor SMD 0805 (2012 Metric), square (rectangular) end terminal, IPC_7351 nominal with elongated pad for handsoldering. (Body size source: IPC-SM-782 page 72, https://www.pcb-3d.com/wordpress/wp-content/uploads/ipc-sm-782a_amendment_1_and_2.pdf), generated with kicad-footprint-generator")
 		(tags "resistor handsolder")
@@
 	(footprint "Footprints:QFN50P400X400X100-25N"
 		(layer "F.Cu")
-		(at 107.1 92.8875)
+		(at 108.6875 93.15)
 		(property "Reference" "U1"
 			(at 0.175 -3.635 0)
@@
 	(footprint "Capacitor_SMD:C_0805_2012Metric_Pad1.18x1.45mm_HandSolder"
 		(layer "F.Cu")
-		(at 112.5 81 -90)
+		(at 115.5 81 -90)
 		(descr "Capacitor SMD 0805 (2012 Metric), square (rectangular) end terminal, IPC_7351 nominal with elongated pad for handsoldering. (Body size source: IPC-SM-782 page 76, https://www.pcb-3d.com/wordpress/wp-content/uploads/ipc-sm-782a_amendment_1_and_2.pdf, https://docs.google.com/spreadsheets/d/1BsfQQcO9C6DZCsRaXUlFlo91Tg2WpOkGARC1WS5S8t0/edit?usp=sharing), generated with kicad-footprint-generator")
 		(tags "capacitor handsolder")
@@
 	(footprint "Footprints:BSS138"
 		(layer "F.Cu")
-		(at 100.94 85.55 180)
+		(at 101.94 86.05 180)
 		(property "Reference" "Q2"
 			(at 0.032 -2.4064 0)
@@
 		(net 1)
 	)
+	(segment
+		(start 108.8375 116.501984)
+		(end 108.8375 116.1625)
+		(width 0.25)
+		(layer "F.Cu")
+		(net 10)
+	)
 )

Commit message: pcb
Parts:
- Q1: moved to B.Cu
- moved C11 12.1 mm to (107.5, 87.5)
- moved RIMON1 11.6 mm to (112.5, 87.5)
- moved Q2 8.19 mm to (94.6, 82.5)
- moved C13 7.40 mm to (103.0, 93.3)
- moved C15 7.40 mm to (103.0, 103.0)
- moved C16 7.40 mm to (103.0, 113.5)
- moved R3 7.16 mm to (102.5, 86.5)
- moved RILIM2 6.71 mm to (109.0, 108.5)
- moved RILIM3 6.58 mm to (109.0, 118.0)
- moved RILIM1 6.04 mm to (109.5, 98.0), turned to 90 degrees
- moved RILIM4 5.53 mm to (110.0, 87.5), turned to 90 degrees
- moved R1 4.27 mm to (94.5, 86.5)
- moved U7 3.86 mm to (109.0, 80.5)
- moved C12 3.50 mm to (118.5, 90.9)
- moved C14 3.50 mm to (118.5, 100.5)
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Connections:
- U3 pad 7: Net-(U1-OVP) -> unconnected-(U3-OVP-Pad7)
Routing:
- net GND: track 0.00 -> 74.5 mm
- net Net-(J1-Pin_2): track 0.00 -> 56.9 mm, vias 0 -> 1
- net Net-(J1-Pin_1): track 0.00 -> 39.2 mm
- net Net-(C13-Pad1): track 0.00 -> 33.3 mm
- net Net-(U1-UVLO): track 0.00 -> 15.5 mm
- net Net-(U7-DRV): track 0.00 -> 12.6 mm
- net Net-(U7-B_GATE): track 0.00 -> 12.1 mm
- net Net-(U1-OVP): track 0.00 -> 9.94 mm
- net Net-(U7-ILIM): track 0.00 -> 6.63 mm
- net Net-(U1-IMON): track 0.00 -> 5.41 mm
- net Net-(U1-dVdT): track 0.00 -> 4.91 mm

Commit message: PBC - brian help
Parts:
- moved RILIM3 9.65 mm to (118.5, 116.3), turned to -90 degrees
- moved RILIM2 1.50 mm to (110.2, 109.4)
- moved RILIM1 1.35 mm to (110.4, 99.0)
Routing:
- net Net-(U1-dVdT): track 4.91 -> 75.7 mm, vias 0 -> 4
- net Net-(U1-~{SHDN}): track 0.00 -> 48.6 mm, vias 0 -> 6
- net Net-(U1-IMON): track 5.41 -> 50.3 mm, vias 0 -> 6
- net Net-(U1-UVLO): track 15.5 -> 51.5 mm
- net Net-(U1-OVP): track 9.94 -> 42.4 mm, vias 0 -> 4
- net Net-(U1-PGOOD): track 0.00 -> 22.8 mm, vias 0 -> 2
- net Net-(U7-PGOOD): track 0.00 -> 19.1 mm, vias 0 -> 2
- net Net-(J1-Pin_1): track 39.2 -> 57.1 mm, vias 0 -> 2
- net GND: track 74.5 -> 90.7 mm
- net Net-(U3-ILIM): track 0.34 -> 15.0 mm
- net Net-(U3-PGTH): track 0.00 -> 13.4 mm, vias 0 -> 2
- net Net-(U2-PGOOD): track 0.00 -> 13.1 mm, vias 0 -> 2
- net Net-(D3-A): track 0.00 -> 6.16 mm
- net Net-(U1-ILIM): track 0.00 -> 5.61 mm
- net Net-(U2-ILIM): track 0.00 -> 5.29 mm
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- added copper zone on F.Cu, net (none)
- added copper zone on B.Cu, net GND
