File: EFUSE2024/EFUSE2024.kicad_pcb (KiCad board)
At the start: 2 copper layers, 34 parts, among them J1 Conn_01x03_Pin, Q1 CSD19537Q3, Q2 BSS138, U1 TPS26630RGE, U2 TPS26630RGE, U3 TPS26630RGE, U7 TPS26630RGE

Commit message: fixed up PCB
Parts:
- removed C12, C13, C14, C16, C17, C18: 0.1uF, Capacitor_SMD:C_0805_2012Metric_Pad1.18x1.45mm_HandSolder
- Q1: moved to F.Cu
- moved C1 5.80 mm to (94.3, 78.8), turned to 0 degrees
- moved R4 4.82 mm to (124.9, 82.2)
- moved C15 3.57 mm to (104.6, 99.8), turned to 180 degrees
- moved C10 3.01 mm to (115.6, 81.8), turned to 0 degrees
- moved Q1 2.36 mm to (102.4, 78.2), turned to 90 degrees
- moved D1 1.46 mm to (101.2, 72.8)
- moved J1 0.80 mm to (113.4, 73.8)
Connections:
- C15 pad 1: Net-(C13-Pad1) -> Net-(U1-DRV)
- Q1 pad 1: Net-(C13-Pad1) -> Net-(U1-DRV)
- Q1 pad 2: Net-(C13-Pad1) -> Net-(U1-DRV)
- Q1 pad 3: Net-(C13-Pad1) -> Net-(U1-DRV)
- Q1 pad 4: Net-(U7-B_GATE) -> Net-(U1-B_GATE)
- Q2 pad 1: Net-(U7-DRV) -> Net-(U1-DRV)
- Q2 pad 2: Net-(U7-B_GATE) -> Net-(U1-B_GATE)
- R7 pad 1: Net-(U3-PGTH) -> Net-(U3-PGOOD)
- U1 pad 1: Net-(C13-Pad1) -> Net-(U1-DRV)
- U1 pad 2: Net-(C13-Pad1) -> Net-(U1-DRV)
- U1 pad 3: unconnected-(U1-B_GATE-Pad3) -> Net-(U1-B_GATE)
- U1 pad 4: unconnected-(U1-DRV-Pad4) -> Net-(U1-DRV)
- U2 pad 1: Net-(C13-Pad1) -> Net-(U1-DRV)
- U2 pad 2: Net-(C13-Pad1) -> Net-(U1-DRV)
- U2 pad 3: unconnected-(U2-B_GATE-Pad3) -> Net-(U1-B_GATE)
- U2 pad 4: unconnected-(U2-DRV-Pad4) -> Net-(U1-DRV)
- U3 pad 1: Net-(C13-Pad1) -> Net-(U1-DRV)
- U3 pad 15: Net-(U3-PGTH) -> unconnected-(U3-PGTH-Pad15)
- U3 pad 16: unconnected-(U3-PGOOD-Pad16) -> Net-(U3-PGOOD)
- U3 pad 2: Net-(C13-Pad1) -> Net-(U1-DRV)
- U3 pad 3: unconnected-(U3-B_GATE-Pad3) -> Net-(U1-B_GATE)
- U3 pad 4: unconnected-(U3-DRV-Pad4) -> Net-(U1-DRV)
- U3 pad 7: unconnected-(U3-OVP-Pad7) -> Net-(U1-OVP)
- U7 pad 1: Net-(C13-Pad1) -> Net-(U1-DRV)
- U7 pad 2: Net-(C13-Pad1) -> Net-(U1-DRV)
- U7 pad 3: Net-(U7-B_GATE) -> Net-(U1-B_GATE)
- U7 pad 4: Net-(U7-DRV) -> Net-(U1-DRV)
Routing:
- net GND: track 90.7 -> 0.34 mm, vias 0 -> 76
- net Net-(U1-B_GATE): track 0.00 -> 67.1 mm, vias 0 -> 7
- net Net-(U1-DRV): track 0.00 -> 56.7 mm, vias 0 -> 14
- net Net-(J1-Pin_1): track 57.1 -> 0.97 mm, vias 2 -> 0
- net Net-(J1-Pin_2): track 56.9 -> 105.7 mm, vias 1 -> 8
- net Net-(U1-dVdT): track 75.7 -> 39.4 mm
- net Net-(C13-Pad1): track 35.6 -> 0.00 mm
- net Net-(U1-UVLO): track 51.5 -> 70.3 mm, vias 0 -> 5
- net Net-(U3-PGTH): track 13.4 -> 0.00 mm, vias 2 -> 0
- net Net-(U1-~{SHDN}): track 48.6 -> 35.5 mm, vias 6 -> 4
- net Net-(U3-PGOOD): track 0.00 -> 13.0 mm, vias 0 -> 2
- net Net-(U7-DRV): track 12.6 -> 0.00 mm
- net Net-(U7-B_GATE): track 12.1 -> 0.00 mm
- net Net-(U1-PGOOD): track 22.8 -> 13.0 mm
- net Net-(U7-PGOOD): track 19.1 -> 13.7 mm
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- added copper zone on F.Cu, net GND
- added copper zone on F.Cu, net Net-(J1-Pin_1)
- added copper zone on F.Cu, net Net-(J1-Pin_2)
- added copper zone on F.Cu, net Net-(U1-DRV)
- removed copper zone on F.Cu, net (none)
Other:
- board outline added: 40 x 50 mm
- board text added: "GND"
- board text added: "IN"
- board text added: "OUT"

Commit message: updates
Connections:
- C15 pad 1: Net-(U1-DRV) -> Net-(C15-Pad1)
- Q1 pad 1: Net-(U1-DRV) -> Net-(C15-Pad1)
- Q1 pad 2: Net-(U1-DRV) -> Net-(C15-Pad1)
- Q1 pad 3: Net-(U1-DRV) -> Net-(C15-Pad1)
- U1 pad 1: Net-(U1-DRV) -> Net-(C15-Pad1)
- U1 pad 2: Net-(U1-DRV) -> Net-(C15-Pad1)
- U2 pad 1: Net-(U1-DRV) -> Net-(C15-Pad1)
- U2 pad 2: Net-(U1-DRV) -> Net-(C15-Pad1)
- U3 pad 1: Net-(U1-DRV) -> Net-(C15-Pad1)
- U3 pad 2: Net-(U1-DRV) -> Net-(C15-Pad1)
- U7 pad 1: Net-(U1-DRV) -> Net-(C15-Pad1)
- U7 pad 2: Net-(U1-DRV) -> Net-(C15-Pad1)
Routing:
- net Net-(U1-DRV): track 56.7 -> 68.3 mm, vias 14 -> 8
- net Net-(U1-dVdT): track 39.4 -> 40.7 mm
- net Net-(J1-Pin_2): track 105.7 -> 106.3 mm
- net GND: vias 76 -> 70
- added copper zone on F.Cu, net Net-(C15-Pad1)
- removed copper zone on F.Cu, net Net-(U1-DRV)
Other:
- board text added: "EFUSE V1 - 2024"

Commit message: updates
Parts:
- moved C15 1.81 mm to (102.8, 99.6)
Routing:
- net Net-(U1-IMON): track 52.9 -> 63.6 mm
- net Net-(U1-dVdT): track 40.7 -> 48.8 mm
- net Net-(U1-OVP): track 44.9 -> 49.9 mm
- net Net-(U1-B_GATE): track 67.0 -> 71.2 mm
- net Net-(U1-~{SHDN}): track 35.5 -> 38.7 mm
- net Net-(J1-Pin_2): track 106.3 -> 109.2 mm, vias 8 -> 6
- net Net-(U1-DRV): track 68.3 -> 70.3 mm, vias 8 -> 6
- net Net-(U1-UVLO): track 70.2 -> 71.9 mm, vias 5 -> 7
- net GND: vias 70 -> 54

Commit message: adding gerber files
Parts:
- renumbered C11 to C1, C1 to C2, C10 to C3, C15 to C4, D5 to D3, D3 to D4, D4 to D5, R7 to R5, R5 to R7, RILIM4 to RILIM1, RILIM1 to RILIM2, RILIM2 to RILIM3, RILIM3 to RILIM4, U7 to U1, U1 to U2, U2 to U3, U3 to U4

Commit message: final update
Parts:
- removed C2: 1uF, Capacitor_SMD:C_0805_2012Metric_Pad1.18x1.45mm_HandSolder
- removed C3, C4: 0.1uF, Capacitor_SMD:C_0805_2012Metric_Pad1.18x1.45mm_HandSolder
- added C10: 0.1uF, Capacitor_SMD:C_0805_2012Metric_Pad1.18x1.45mm_HandSolder, F.Cu at (117.6, 81.8)
- added C11: 0.1uF, Capacitor_SMD:C_0805_2012Metric_Pad1.18x1.45mm_HandSolder, F.Cu at (107.3, 87.4)
- added C15: 0.1uF, Capacitor_SMD:C_0805_2012Metric_Pad1.18x1.45mm_HandSolder, F.Cu at (102.8, 99.8)
- added JP1: Jumper_2_Bridged, Jumper:SolderJumper-2_P1.3mm_Bridged2Bar_Pad1.0x1.5mm, F.Cu at (112.7, 108.7)
- added JP2: Jumper_2_Bridged, Jumper:SolderJumper-2_P1.3mm_Bridged2Bar_Pad1.0x1.5mm, F.Cu at (113.7, 117.0)
- added JP3: Jumper_2_Bridged, Jumper:SolderJumper-2_P1.3mm_Bridged2Bar_Pad1.0x1.5mm, F.Cu at (113.2, 96.2)
- added JP4: Jumper_2_Bridged, Jumper:SolderJumper-2_P1.3mm_Bridged2Bar_Pad1.0x1.5mm, F.Cu at (113.3, 83.8)
- C1: value 0.1uF -> 1uF
- D1: value SMCJ36CA -> DIOM6859X262N
- Q2: value BSS138 -> SOT95P240X111-3N
- moved C1 15.7 mm to (94.4, 78.8), turned to 0 degrees
- moved RILIM4 2.24 mm to (118.1, 118.5), turned to 0 degrees
Connections:
- C1 pad 1: Net-(U1-dVdT) -> Net-(J1-Pin_2)
- Q1 pad 1: Net-(C15-Pad1) -> Net-(U1-DRV)
- Q1 pad 2: Net-(C15-Pad1) -> Net-(U1-DRV)
- Q1 pad 3: Net-(C15-Pad1) -> Net-(U1-DRV)
- U1 pad 1: Net-(C15-Pad1) -> Net-(U1-DRV)
- U1 pad 11: GND -> Net-(JP4-B)
- U1 pad 2: Net-(C15-Pad1) -> Net-(U1-DRV)
- U2 pad 1: Net-(C15-Pad1) -> Net-(U1-DRV)
- U2 pad 11: GND -> Net-(JP3-B)
- U2 pad 2: Net-(C15-Pad1) -> Net-(U1-DRV)
- U3 pad 1: Net-(C15-Pad1) -> Net-(U1-DRV)
- U3 pad 11: GND -> Net-(JP1-B)
- U3 pad 2: Net-(C15-Pad1) -> Net-(U1-DRV)
- U4 pad 1: Net-(C15-Pad1) -> Net-(U1-DRV)
- U4 pad 11: GND -> Net-(JP2-B)
- U4 pad 2: Net-(C15-Pad1) -> Net-(U1-DRV)
Routing:
- net Net-(JP3-B): track 0.00 -> 5.21 mm
- net Net-(JP4-B): track 0.00 -> 5.03 mm
- net Net-(JP1-B): track 0.00 -> 4.62 mm
- net Net-(JP2-B): track 0.00 -> 4.28 mm
- net Net-(U4-ILIM): track 11.0 -> 9.51 mm
- net GND: track 0.34 -> 0.00 mm, vias 54 -> 58
- added copper zone on F.Cu, net Net-(U1-DRV)
- removed copper zone on F.Cu, net Net-(C15-Pad1)

Commit message: update
Parts:
- D2, D3, D4, D5: footprint LED_SMD:LED_2512_6332Metric_Pad1.52x3.35mm_HandSolder -> LED_SMD:LED_1206_3216Metric_Pad1.42x1.75mm_HandSolder
- moved RILIM4 0.30 mm to (118.1, 118.2)
Routing:
- net Net-(D5-A): track 4.50 -> 5.12 mm
- net Net-(D4-A): track 6.16 -> 5.54 mm
- net Net-(D3-A): track 5.00 -> 4.38 mm
- net GND: vias 58 -> 41
